Commit message: train_3axis.py run ok, but not workking properly

File: robot_description/3dof_cartesian_robot.urdf (robot description, URDF)
Before this commit: robot 3dof_cartesian_robot, 4 links, 3 joints
Links:
- link base_link: mass None -> 1.0
- link link_x: mass None -> 0.5
- link link_y: mass None -> 0.5
- link link_z: mass None -> 0.5

Commit message: urdf visual tag added

File: robot_description/3dof_cartesian_robot.urdf (robot description, URDF)
Before this commit: robot 3dof_cartesian_robot, 4 links, 3 joints
Links:
- link base_link: geometry visual box size=0.1 0.1 0.1
- link link_x: mass 0.5 -> 1.0; geometry visual box size=1.0 0.03 0.03
- link link_y: mass 0.5 -> 1.0; geometry visual box size=0.03 1.0 0.03
- link link_z: mass 0.5 -> 1.0; geometry visual box size=0.03 0.03 1.0
Joints:
- joint joint_x: origin (none) -> xyz=0 0 0 rpy=0 0 0
- joint joint_y: origin (none) -> xyz=0 0 0 rpy=0 0 0
- joint joint_z: origin (none) -> xyz=0 0 0 rpy=0 0 0

Commit message: env set OK

File: robot_description/3dof_cartesian_robot.urdf (robot description, URDF)
Before this commit: robot 3dof_cartesian_robot, 4 links, 3 joints
Links:
- link base_link: mass 1.0 -> None
- link link_x: mass 1.0 -> None
- link link_y: mass 1.0 -> None
- link link_z: mass 1.0 -> None
Joints:
- joint joint_x: origin xyz=0 0 0 rpy=0 0 0 -> xyz=0 0.5 0 rpy=0 0 0; parent base_link -> link_y
- joint joint_y: origin xyz=0 0 0 rpy=0 0 0 -> xyz=0 0 0.5 rpy=0 0 0; parent link_x -> link_z
- joint joint_z: limit lower=0 upper=1 effort=100 velocity=0.5 -> lower=0 upper=1 effort=500 velocity=0.5; parent link_y -> base_link

Commit message: add inertia in urdf

File: robot_description/3dof_cartesian_robot.urdf (robot description, URDF)
Before this commit: robot 3dof_cartesian_robot, 4 links, 3 joints
Links:
- added link end_effector, mass 0.1; collision sphere radius=0.05; visual sphere radius=0.05
- link base_link: mass None -> 1.0; geometry collision box size=0.1 0.1 0.1; visual box size=0.1 0.1 0.1
- link link_x: mass None -> 0.5; geometry collision box size=1.0 0.03 0.03; visual box size=1.0 0.03 0.03
- link link_y: mass None -> 0.5; geometry collision box size=0.03 1.0 0.03; visual box size=0.03 1.0 0.03
- link link_z: mass None -> 0.5; geometry collision box size=0.03 0.03 1.0; visual box size=0.03 0.03 1.0
Joints:
- added joint joint_end_effector: type fixed, parent link_x, child end_effector, origin xyz=0.5 0 0 rpy=0 0 0
